Commit message: Add environ

File: project_starter_code/toro.urdf (robot description, URDF)
Before this commit: robot DLR_TORO, 34 links, 33 joints
Links:
- link RL_KOSY_L1: geometry collision capsule a=0.00832896 0.0340227 -0.112749 b=0.00832895 -0.0145192 -0.112749 radius=0.0755809; visual mesh filename=../../../model/toro/meshes/obj/right_lower_hip.stl.obj
- link RL_KOSY_L23: geometry collision capsule a=0 -0.037 0 b=0 0.0 -0.17 radius=0.0764886; visual mesh filename=../../../model/toro/meshes/obj/kuka-link2.stl.obj
- link RL_foot: mass 142.41951000 -> 1.4241951000
- link hip_base: geometry collision capsule a=-0.0177247 -0.134409 -0.117853 b=-0.0177247 0.134409 -0.117853 radius=0.072616; visual mesh filename=../../../model/toro/meshes/obj/upper_hip.stl.obj
- link ra_link5: geometry collision capsule a=9.5357e-06 -1.3717e-06 0.103513 b=-4.69339e-05 7.35371e-06 0.206594 radius=0.0662048; visual mesh filename=../../../model/toro/meshes/obj/va_right_lower_arm.stl.obj
Joints:
- joint j1: limit lower=-1.5708 upper=0.7854 effort=176 velocity=1.9199 -> lower=-1.5708 upper=0.7854 effort=1760 velocity=19.199
- joint j10: limit lower=-1.8326 upper=1.8326 effort=165 velocity=3.0718 -> lower=0 upper=1.8326 effort=1650 velocity=30.718
- joint j11: limit lower=-0.3403 upper=0.3403 effort=50 velocity=2.0944 -> lower=-0.3403 upper=0.3403 effort=500 velocity=20.944
- joint j12: limit lower=-0.7854 upper=0.7854 effort=165 velocity=3.0718 -> lower=-0.7854 upper=0.7854 effort=1650 velocity=30.718
- joint j13: limit lower=-2.0944 upper=2.0944 effort=100 velocity=2.7402 -> lower=-2.0944 upper=2.0944 effort=1000 velocity=27.402
- joint j14: limit lower=-2.0944 upper=2.0944 effort=100 velocity=2.7402 -> lower=-2.0944 upper=2.0944 effort=1000 velocity=27.402
- joint j15: limit lower=-0.2618 upper=3.1416 effort=100 velocity=2.7402 -> lower=-0.2618 upper=3.1416 effort=1000 velocity=27.402
- joint j16: limit lower=-1.8326 upper=1.8326 effort=40 velocity=2.0944 -> lower=-1.8326 upper=1.8326 effort=400 velocity=20.944
- joint j17: limit lower=0 upper=2.5831 effort=40 velocity=2.0944 -> lower=-1 upper=2.5831 effort=400 velocity=20.944
- joint j18: limit lower=-2.5307 upper=2.0595 effort=40 velocity=2.0944 -> lower=-2.5307 upper=2.0595 effort=400 velocity=20.944
- joint j19: limit lower=-1.8326 upper=1.8326 effort=35 velocity=2.0944 -> lower=-1.8326 upper=1.8326 effort=350 velocity=20.944
- joint j2: limit lower=-2.0071 upper=1.5708 effort=100 velocity=2.7402 -> lower=-2.0071 upper=1.5708 effort=1000 velocity=27.402
- joint j20: limit lower=-2.0944 upper=2.0944 effort=100 velocity=2.7402 -> lower=-2.0944 upper=2.0944 effort=1000 velocity=27.402
- joint j21: limit lower=-0.2618 upper=3.1416 effort=100 velocity=2.7402 -> lower=-0.2618 upper=3.1416 effort=1000 velocity=27.402
- joint j22: limit lower=-1.8326 upper=1.8326 effort=40 velocity=2.0944 -> lower=-1.8326 upper=1.8326 effort=400 velocity=20.944
- joint j23: limit lower=0 upper=2.5831 effort=40 velocity=2.0944 -> lower=-1 upper=2.5831 effort=400 velocity=20.944
- joint j24: limit lower=-2.5307 upper=2.0595 effort=40 velocity=2.0944 -> lower=-2.5307 upper=2.0595 effort=400 velocity=20.944
- joint j25: limit lower=-1.8326 upper=1.8326 effort=40 velocity=2.0944 -> lower=-1.8326 upper=1.8326 effort=400 velocity=20.944
- joint j26: limit lower=-1.5708 upper=1.5708 effort=8.4 velocity=4.7124 -> lower=-1.5708 upper=1.5708 effort=84 velocity=47.124
- joint j27: limit lower=-0.5236 upper=1.5708 effort=8.4 velocity=4.7124 -> lower=-0.5236 upper=1.5708 effort=84 velocity=47.124
- joint j3: limit lower=-2.0944 upper=2.0944 effort=100 velocity=2.7402 -> lower=-2.0944 upper=2.0944 effort=1000 velocity=27.402
- joint j4: limit lower=-1.8326 upper=1.8326 effort=165 velocity=3.0718 -> lower=0 upper=1.8326 effort=1650 velocity=30.718
- joint j5: limit lower=-0.3403 upper=0.3403 effort=50 velocity=2.0944 -> lower=-0.3403 upper=0.3403 effort=500 velocity=20.944
- joint j6: limit lower=-0.7804 upper=0.7804 effort=165 velocity=3.0718 -> lower=-0.7854 upper=0.7854 effort=1650 velocity=30.718
- joint j7: limit lower=-0.7804 upper=1.5708 effort=176 velocity=1.9199 -> lower=-0.7804 upper=1.5708 effort=1760 velocity=19.199
- joint j8: limit lower=-2.0071 upper=1.5708 effort=100 velocity=2.7402 -> lower=-2.0071 upper=1.5708 effort=1000 velocity=27.402
- joint j9: limit lower=-2.0944 upper=2.0944 effort=100 velocity=2.7402 -> lower=-2.0944 upper=2.0944 effort=1000 velocity=27.402
